Commit message: Add files via upload

File: moroder.urdf (robot description, URDF)
Before this commit: robot moroder, 22 links, 21 joints
Links:
- link end_effectorBL: mass 0.022 -> 0.002
- link end_effectorBR: mass 0.022 -> 0.002
- link end_effectorFL: mass 0.022 -> 0.002
- link end_effectorFR: mass 0.022 -> 0.002
- link head: mass 0.001 -> 0.0001
- link tibiaBL: geometry collision cylinder length=0.06 radius=0.00625; visual cylinder length=0.06 radius=0.00625
- link tibiaBR: geometry collision cylinder length=0.06 radius=0.00625; visual cylinder length=0.06 radius=0.00625
- link tibiaFL: geometry collision cylinder length=0.06 radius=0.00625; visual cylinder length=0.06 radius=0.00625
- link tibiaFR: geometry collision cylinder length=0.06 radius=0.00625; visual cylinder length=0.06 radius=0.00625
Joints:
- joint coxa_linkBL: limit lower=-0.1 upper=0.1 effort=999 velocity=5,233333333 -> lower=-0.000 upper=0.000 effort=999 velocity=5,233333333
- joint coxa_linkBR: limit lower=-0.1 upper=0.1 effort=999 velocity=5,233333333 -> lower=-0.000 upper=0.000 effort=999 velocity=5,233333333
- joint coxa_linkFL: limit lower=-0.1 upper=0.1 effort=999 velocity=5,233333333 -> lower=-0.000 upper=0.000 effort=999 velocity=5,233333333
- joint coxa_linkFR: limit lower=-0.1 upper=0.1 effort=999 velocity=5,233333333 -> lower=-0.000 upper=0.000 effort=999 velocity=5,233333333
- joint pauldron_linkBL: limit lower=-1 upper=1 effort=999 velocity=5,233333333 -> lower=-1.0472 upper=1.0472 effort=999 velocity=5,233333333
- joint pauldron_linkBR: limit lower=-1 upper=1 effort=999 velocity=5,233333333 -> lower=-1.0472 upper=1.0472 effort=999 velocity=5,233333333
- joint pauldron_linkFL: limit lower=-1 upper=1 effort=999 velocity=5,233333333 -> lower=-1.0472 upper=1.0472 effort=999 velocity=5,233333333
- joint pauldron_linkFR: limit lower=-1 upper=1 effort=999 velocity=5,233333333 -> lower=-1.0472 upper=1.0472 effort=999 velocity=5,233333333
- joint tibia_linkBL: limit lower=-0 upper=2 effort=999 velocity=5,233333333 -> lower=0 upper=2.0944 effort=999 velocity=5,233333333
- joint tibia_linkBR: limit lower=-0 upper=2 effort=999 velocity=5,233333333 -> lower=0 upper=2.0944 effort=999 velocity=5,233333333
- joint tibia_linkFL: limit lower=-0 upper=2 effort=999 velocity=5,233333333 -> lower=0 upper=2.0944 effort=999 velocity=5,233333333
- joint tibia_linkFR: limit lower=-0 upper=2 effort=999 velocity=5,233333333 -> lower=0 upper=2.0944 effort=999 velocity=5,233333333
